Commit message: Add little_force_sensor_1 pads: 80 sensors (8x10 layout)
- Added 80 sensor pads to little_force_sensor_1 with 8x10 layout
- Specifications: 1.2mm×1.2mm×0.6mm, 15g trigger, 20N range, 200FPS
- Color: yellow for visual identification
- Total system now has 632 contact points across 8 sensor areas
- Verified alignment with little_force_sensor_1 orientation (rpy=0 0 0)
- Successfully converted to USD format (20.8MB)
- Updated Isaac Lab YAML configuration

File: cabinet_sensor_project/inspire_hand_with_sensors/urdf/inspire_hand_processed_with_pads_before_little1.urdf (robot description, URDF)
Before this commit: robot inspire_hand_with_sensors, 663 links, 662 joints
Links:
- removed link little_sensor_1_pad_001
- removed link little_sensor_1_pad_002
- removed link little_sensor_1_pad_003
- removed link little_sensor_1_pad_004
- removed link little_sensor_1_pad_005
- removed link little_sensor_1_pad_006
- removed link little_sensor_1_pad_007
- removed link little_sensor_1_pad_008
- removed link little_sensor_1_pad_009
- removed link little_sensor_1_pad_010
- removed link little_sensor_1_pad_011
- removed link little_sensor_1_pad_012
- removed link little_sensor_1_pad_013
- removed link little_sensor_1_pad_014
- removed link little_sensor_1_pad_015
- removed link little_sensor_1_pad_016
- removed link little_sensor_1_pad_017
- removed link little_sensor_1_pad_018
- removed link little_sensor_1_pad_019
- removed link little_sensor_1_pad_020
- removed link little_sensor_1_pad_021
- removed link little_sensor_1_pad_022
- removed link little_sensor_1_pad_023
- removed link little_sensor_1_pad_024
- removed link little_sensor_1_pad_025
- removed link little_sensor_1_pad_026
- removed link little_sensor_1_pad_027
- removed link little_sensor_1_pad_028
- removed link little_sensor_1_pad_029
- removed link little_sensor_1_pad_030
- removed link little_sensor_1_pad_031
- removed link little_sensor_1_pad_032
- removed link little_sensor_1_pad_033
- removed link little_sensor_1_pad_034
- removed link little_sensor_1_pad_035
- removed link little_sensor_1_pad_036
- removed link little_sensor_1_pad_037
- removed link little_sensor_1_pad_038
- removed link little_sensor_1_pad_039
- removed link little_sensor_1_pad_040
- removed link little_sensor_1_pad_041
- removed link little_sensor_1_pad_042
- removed link little_sensor_1_pad_043
- removed link little_sensor_1_pad_044
- removed link little_sensor_1_pad_045
- removed link little_sensor_1_pad_046
- removed link little_sensor_1_pad_047
- removed link little_sensor_1_pad_048
- removed link little_sensor_1_pad_049
- removed link little_sensor_1_pad_050
- removed link little_sensor_1_pad_051
- removed link little_sensor_1_pad_052
- removed link little_sensor_1_pad_053
- removed link little_sensor_1_pad_054
- removed link little_sensor_1_pad_055
- removed link little_sensor_1_pad_056
- removed link little_sensor_1_pad_057
- removed link little_sensor_1_pad_058
- removed link little_sensor_1_pad_059
- removed link little_sensor_1_pad_060
- removed link little_sensor_1_pad_061
- removed link little_sensor_1_pad_062
- removed link little_sensor_1_pad_063
- removed link little_sensor_1_pad_064
- removed link little_sensor_1_pad_065
- removed link little_sensor_1_pad_066
- removed link little_sensor_1_pad_067
- removed link little_sensor_1_pad_068
- removed link little_sensor_1_pad_069
- removed link little_sensor_1_pad_070
- removed link little_sensor_1_pad_071
- removed link little_sensor_1_pad_072
- removed link little_sensor_1_pad_073
- removed link little_sensor_1_pad_074
- removed link little_sensor_1_pad_075
- removed link little_sensor_1_pad_076
- removed link little_sensor_1_pad_077
- removed link little_sensor_1_pad_078
- removed link little_sensor_1_pad_079
- removed link little_sensor_1_pad_080
Joints:
- removed joint little_sensor_1_pad_001_joint
- removed joint little_sensor_1_pad_002_joint
- removed joint little_sensor_1_pad_003_joint
- removed joint little_sensor_1_pad_004_joint
- removed joint little_sensor_1_pad_005_joint
- removed joint little_sensor_1_pad_006_joint
- removed joint little_sensor_1_pad_007_joint
- removed joint little_sensor_1_pad_008_joint
- removed joint little_sensor_1_pad_009_joint
- removed joint little_sensor_1_pad_010_joint
- removed joint little_sensor_1_pad_011_joint
- removed joint little_sensor_1_pad_012_joint
- removed joint little_sensor_1_pad_013_joint
- removed joint little_sensor_1_pad_014_joint
- removed joint little_sensor_1_pad_015_joint
- removed joint little_sensor_1_pad_016_joint
- removed joint little_sensor_1_pad_017_joint
- removed joint little_sensor_1_pad_018_joint
- removed joint little_sensor_1_pad_019_joint
- removed joint little_sensor_1_pad_020_joint
- removed joint little_sensor_1_pad_021_joint
- removed joint little_sensor_1_pad_022_joint
- removed joint little_sensor_1_pad_023_joint
- removed joint little_sensor_1_pad_024_joint
- removed joint little_sensor_1_pad_025_joint
- removed joint little_sensor_1_pad_026_joint
- removed joint little_sensor_1_pad_027_joint
- removed joint little_sensor_1_pad_028_joint
- removed joint little_sensor_1_pad_029_joint
- removed joint little_sensor_1_pad_030_joint
- removed joint little_sensor_1_pad_031_joint
- removed joint little_sensor_1_pad_032_joint
- removed joint little_sensor_1_pad_033_joint
- removed joint little_sensor_1_pad_034_joint
- removed joint little_sensor_1_pad_035_joint
- removed joint little_sensor_1_pad_036_joint
- removed joint little_sensor_1_pad_037_joint
- removed joint little_sensor_1_pad_038_joint
- removed joint little_sensor_1_pad_039_joint
- removed joint little_sensor_1_pad_040_joint
- removed joint little_sensor_1_pad_041_joint
- removed joint little_sensor_1_pad_042_joint
- removed joint little_sensor_1_pad_043_joint
- removed joint little_sensor_1_pad_044_joint
- removed joint little_sensor_1_pad_045_joint
- removed joint little_sensor_1_pad_046_joint
- removed joint little_sensor_1_pad_047_joint
- removed joint little_sensor_1_pad_048_joint
- removed joint little_sensor_1_pad_049_joint
- removed joint little_sensor_1_pad_050_joint
- removed joint little_sensor_1_pad_051_joint
- removed joint little_sensor_1_pad_052_joint
- removed joint little_sensor_1_pad_053_joint
- removed joint little_sensor_1_pad_054_joint
- removed joint little_sensor_1_pad_055_joint
- removed joint little_sensor_1_pad_056_joint
- removed joint little_sensor_1_pad_057_joint
- removed joint little_sensor_1_pad_058_joint
- removed joint little_sensor_1_pad_059_joint
- removed joint little_sensor_1_pad_060_joint
- removed joint little_sensor_1_pad_061_joint
- removed joint little_sensor_1_pad_062_joint
- removed joint little_sensor_1_pad_063_joint
- removed joint little_sensor_1_pad_064_joint
- removed joint little_sensor_1_pad_065_joint
- removed joint little_sensor_1_pad_066_joint
- removed joint little_sensor_1_pad_067_joint
- removed joint little_sensor_1_pad_068_joint
- removed joint little_sensor_1_pad_069_joint
- removed joint little_sensor_1_pad_070_joint
- removed joint little_sensor_1_pad_071_joint
- removed joint little_sensor_1_pad_072_joint
- removed joint little_sensor_1_pad_073_joint
- removed joint little_sensor_1_pad_074_joint
- removed joint little_sensor_1_pad_075_joint
- removed joint little_sensor_1_pad_076_joint
- removed joint little_sensor_1_pad_077_joint
- removed joint little_sensor_1_pad_078_joint
- removed joint little_sensor_1_pad_079_joint
- removed joint little_sensor_1_pad_080_joint
