Commit message: Add thumb_force_sensor_2 pads (2x4) and convert to USD
- Added 8 sensor pads to thumb_force_sensor_2 in 2x4 grid layout
- Each pad: 1.2mm×1.2mm×0.6mm, 15g trigger, 20N max, 200FPS
- Created conversion script convert_urdf_to_usd_with_thumb2_pads.py
- Generated USD and YAML files with Isaac Lab configuration
- Total sensors: 220 contact points (112 palm + 96 thumb1 + 8 thumb2 + 4 force)
- Excluded large USDA file from repository

File: cabinet_sensor_project/inspire_hand_with_sensors/urdf/inspire_hand_processed_with_pads.urdf (robot description, URDF)
Before this commit: robot inspire_hand_with_sensors, 239 links, 238 joints
Links:
- added link thumb_sensor_2_pad_001, mass 0.000001; collision box size=0.001200 0.001200 0.000600; visual box size=0.001200 0.001200 0.000600
- added link thumb_sensor_2_pad_002, mass 0.000001; collision box size=0.001200 0.001200 0.000600; visual box size=0.001200 0.001200 0.000600
- added link thumb_sensor_2_pad_003, mass 0.000001; collision box size=0.001200 0.001200 0.000600; visual box size=0.001200 0.001200 0.000600
- added link thumb_sensor_2_pad_004, mass 0.000001; collision box size=0.001200 0.001200 0.000600; visual box size=0.001200 0.001200 0.000600
- added link thumb_sensor_2_pad_005, mass 0.000001; collision box size=0.001200 0.001200 0.000600; visual box size=0.001200 0.001200 0.000600
- added link thumb_sensor_2_pad_006, mass 0.000001; collision box size=0.001200 0.001200 0.000600; visual box size=0.001200 0.001200 0.000600
- added link thumb_sensor_2_pad_007, mass 0.000001; collision box size=0.001200 0.001200 0.000600; visual box size=0.001200 0.001200 0.000600
- added link thumb_sensor_2_pad_008, mass 0.000001; collision box size=0.001200 0.001200 0.000600; visual box size=0.001200 0.001200 0.000600
Joints:
- added joint thumb_sensor_2_pad_001_joint: type fixed, parent thumb_force_sensor_2, child thumb_sensor_2_pad_001, origin xyz=-0.000600 -0.001800 0.000300 rpy=0 0 0
- added joint thumb_sensor_2_pad_002_joint: type fixed, parent thumb_force_sensor_2, child thumb_sensor_2_pad_002, origin xyz=-0.000600 -0.000600 0.000300 rpy=0 0 0
- added joint thumb_sensor_2_pad_003_joint: type fixed, parent thumb_force_sensor_2, child thumb_sensor_2_pad_003, origin xyz=-0.000600 0.000600 0.000300 rpy=0 0 0
- added joint thumb_sensor_2_pad_004_joint: type fixed, parent thumb_force_sensor_2, child thumb_sensor_2_pad_004, origin xyz=-0.000600 0.001800 0.000300 rpy=0 0 0
- added joint thumb_sensor_2_pad_005_joint: type fixed, parent thumb_force_sensor_2, child thumb_sensor_2_pad_005, origin xyz=0.000600 -0.001800 0.000300 rpy=0 0 0
- added joint thumb_sensor_2_pad_006_joint: type fixed, parent thumb_force_sensor_2, child thumb_sensor_2_pad_006, origin xyz=0.000600 -0.000600 0.000300 rpy=0 0 0
- added joint thumb_sensor_2_pad_007_joint: type fixed, parent thumb_force_sensor_2, child thumb_sensor_2_pad_007, origin xyz=0.000600 0.000600 0.000300 rpy=0 0 0
- added joint thumb_sensor_2_pad_008_joint: type fixed, parent thumb_force_sensor_2, child thumb_sensor_2_pad_008, origin xyz=0.000600 0.001800 0.000300 rpy=0 0 0
