Commit message: 🔧 Add Little2 sensor pads: 80 pads (8×10) - Total: 952 sensor pads
- Added 80 little_sensor_2_pad_XXX links and joints to little_force_sensor_2
- Little2 sensor pads use 8×10 grid layout for consistency with other finger sensors
- Updated USD conversion script with Little2 sensor configuration
- Updated Isaac Lab configuration with little_sensor_2_pads section
- Total sensor pads: 952 (Palm:112, Thumb1:96, Thumb2:8, Thumb3:96, Index1:80, Index2:80, Middle1:80, Middle2:80, Ring1:80, Ring2:80, Little1:80, Little2:80)
- All finger sensors now have consistent 8×10 layouts (except Middle1: 10×8)
- Little2 pads: light_yellow color, 1.2×1.2×0.6mm size

File: cabinet_sensor_project/inspire_hand_with_sensors/urdf/inspire_hand_processed_with_pads.urdf (robot description, URDF)
Before this commit: robot inspire_hand_with_sensors, 903 links, 902 joints
Links:
- added link little_sensor_2_pad_001, mass 0.000001; collision box size=0.001200 0.001200 0.000600; visual box size=0.001200 0.001200 0.000600
- added link little_sensor_2_pad_002, mass 0.000001; collision box size=0.001200 0.001200 0.000600; visual box size=0.001200 0.001200 0.000600
- added link little_sensor_2_pad_003, mass 0.000001; collision box size=0.001200 0.001200 0.000600; visual box size=0.001200 0.001200 0.000600
- added link little_sensor_2_pad_004, mass 0.000001; collision box size=0.001200 0.001200 0.000600; visual box size=0.001200 0.001200 0.000600
- added link little_sensor_2_pad_005, mass 0.000001; collision box size=0.001200 0.001200 0.000600; visual box size=0.001200 0.001200 0.000600
- added link little_sensor_2_pad_006, mass 0.000001; collision box size=0.001200 0.001200 0.000600; visual box size=0.001200 0.001200 0.000600
- added link little_sensor_2_pad_007, mass 0.000001; collision box size=0.001200 0.001200 0.000600; visual box size=0.001200 0.001200 0.000600
- added link little_sensor_2_pad_008, mass 0.000001; collision box size=0.001200 0.001200 0.000600; visual box size=0.001200 0.001200 0.000600
- added link little_sensor_2_pad_009, mass 0.000001; collision box size=0.001200 0.001200 0.000600; visual box size=0.001200 0.001200 0.000600
- added link little_sensor_2_pad_010, mass 0.000001; collision box size=0.001200 0.001200 0.000600; visual box size=0.001200 0.001200 0.000600
- added link little_sensor_2_pad_011, mass 0.000001; collision box size=0.001200 0.001200 0.000600; visual box size=0.001200 0.001200 0.000600
- added link little_sensor_2_pad_012, mass 0.000001; collision box size=0.001200 0.001200 0.000600; visual box size=0.001200 0.001200 0.000600
- added link little_sensor_2_pad_013, mass 0.000001; collision box size=0.001200 0.001200 0.000600; visual box size=0.001200 0.001200 0.000600
- added link little_sensor_2_pad_014, mass 0.000001; collision box size=0.001200 0.001200 0.000600; visual box size=0.001200 0.001200 0.000600
- added link little_sensor_2_pad_015, mass 0.000001; collision box size=0.001200 0.001200 0.000600; visual box size=0.001200 0.001200 0.000600
- added link little_sensor_2_pad_016, mass 0.000001; collision box size=0.001200 0.001200 0.000600; visual box size=0.001200 0.001200 0.000600
- added link little_sensor_2_pad_017, mass 0.000001; collision box size=0.001200 0.001200 0.000600; visual box size=0.001200 0.001200 0.000600
- added link little_sensor_2_pad_018, mass 0.000001; collision box size=0.001200 0.001200 0.000600; visual box size=0.001200 0.001200 0.000600
- added link little_sensor_2_pad_019, mass 0.000001; collision box size=0.001200 0.001200 0.000600; visual box size=0.001200 0.001200 0.000600
- added link little_sensor_2_pad_020, mass 0.000001; collision box size=0.001200 0.001200 0.000600; visual box size=0.001200 0.001200 0.000600
- added link little_sensor_2_pad_021, mass 0.000001; collision box size=0.001200 0.001200 0.000600; visual box size=0.001200 0.001200 0.000600
- added link little_sensor_2_pad_022, mass 0.000001; collision box size=0.001200 0.001200 0.000600; visual box size=0.001200 0.001200 0.000600
- added link little_sensor_2_pad_023, mass 0.000001; collision box size=0.001200 0.001200 0.000600; visual box size=0.001200 0.001200 0.000600
- added link little_sensor_2_pad_024, mass 0.000001; collision box size=0.001200 0.001200 0.000600; visual box size=0.001200 0.001200 0.000600
- added link little_sensor_2_pad_025, mass 0.000001; collision box size=0.001200 0.001200 0.000600; visual box size=0.001200 0.001200 0.000600
- added link little_sensor_2_pad_026, mass 0.000001; collision box size=0.001200 0.001200 0.000600; visual box size=0.001200 0.001200 0.000600
- added link little_sensor_2_pad_027, mass 0.000001; collision box size=0.001200 0.001200 0.000600; visual box size=0.001200 0.001200 0.000600
- added link little_sensor_2_pad_028, mass 0.000001; collision box size=0.001200 0.001200 0.000600; visual box size=0.001200 0.001200 0.000600
- added link little_sensor_2_pad_029, mass 0.000001; collision box size=0.001200 0.001200 0.000600; visual box size=0.001200 0.001200 0.000600
- added link little_sensor_2_pad_030, mass 0.000001; collision box size=0.001200 0.001200 0.000600; visual box size=0.001200 0.001200 0.000600
- added link little_sensor_2_pad_031, mass 0.000001; collision box size=0.001200 0.001200 0.000600; visual box size=0.001200 0.001200 0.000600
- added link little_sensor_2_pad_032, mass 0.000001; collision box size=0.001200 0.001200 0.000600; visual box size=0.001200 0.001200 0.000600
- added link little_sensor_2_pad_033, mass 0.000001; collision box size=0.001200 0.001200 0.000600; visual box size=0.001200 0.001200 0.000600
- added link little_sensor_2_pad_034, mass 0.000001; collision box size=0.001200 0.001200 0.000600; visual box size=0.001200 0.001200 0.000600
- added link little_sensor_2_pad_035, mass 0.000001; collision box size=0.001200 0.001200 0.000600; visual box size=0.001200 0.001200 0.000600
- added link little_sensor_2_pad_036, mass 0.000001; collision box size=0.001200 0.001200 0.000600; visual box size=0.001200 0.001200 0.000600
- added link little_sensor_2_pad_037, mass 0.000001; collision box size=0.001200 0.001200 0.000600; visual box size=0.001200 0.001200 0.000600
- added link little_sensor_2_pad_038, mass 0.000001; collision box size=0.001200 0.001200 0.000600; visual box size=0.001200 0.001200 0.000600
- added link little_sensor_2_pad_039, mass 0.000001; collision box size=0.001200 0.001200 0.000600; visual box size=0.001200 0.001200 0.000600
- added link little_sensor_2_pad_040, mass 0.000001; collision box size=0.001200 0.001200 0.000600; visual box size=0.001200 0.001200 0.000600
- added link little_sensor_2_pad_041, mass 0.000001; collision box size=0.001200 0.001200 0.000600; visual box size=0.001200 0.001200 0.000600
- added link little_sensor_2_pad_042, mass 0.000001; collision box size=0.001200 0.001200 0.000600; visual box size=0.001200 0.001200 0.000600
- added link little_sensor_2_pad_043, mass 0.000001; collision box size=0.001200 0.001200 0.000600; visual box size=0.001200 0.001200 0.000600
- added link little_sensor_2_pad_044, mass 0.000001; collision box size=0.001200 0.001200 0.000600; visual box size=0.001200 0.001200 0.000600
- added link little_sensor_2_pad_045, mass 0.000001; collision box size=0.001200 0.001200 0.000600; visual box size=0.001200 0.001200 0.000600
- added link little_sensor_2_pad_046, mass 0.000001; collision box size=0.001200 0.001200 0.000600; visual box size=0.001200 0.001200 0.000600
- added link little_sensor_2_pad_047, mass 0.000001; collision box size=0.001200 0.001200 0.000600; visual box size=0.001200 0.001200 0.000600
- added link little_sensor_2_pad_048, mass 0.000001; collision box size=0.001200 0.001200 0.000600; visual box size=0.001200 0.001200 0.000600
- added link little_sensor_2_pad_049, mass 0.000001; collision box size=0.001200 0.001200 0.000600; visual box size=0.001200 0.001200 0.000600
- added link little_sensor_2_pad_050, mass 0.000001; collision box size=0.001200 0.001200 0.000600; visual box size=0.001200 0.001200 0.000600
- added link little_sensor_2_pad_051, mass 0.000001; collision box size=0.001200 0.001200 0.000600; visual box size=0.001200 0.001200 0.000600
- added link little_sensor_2_pad_052, mass 0.000001; collision box size=0.001200 0.001200 0.000600; visual box size=0.001200 0.001200 0.000600
- added link little_sensor_2_pad_053, mass 0.000001; collision box size=0.001200 0.001200 0.000600; visual box size=0.001200 0.001200 0.000600
- added link little_sensor_2_pad_054, mass 0.000001; collision box size=0.001200 0.001200 0.000600; visual box size=0.001200 0.001200 0.000600
- added link little_sensor_2_pad_055, mass 0.000001; collision box size=0.001200 0.001200 0.000600; visual box size=0.001200 0.001200 0.000600
- added link little_sensor_2_pad_056, mass 0.000001; collision box size=0.001200 0.001200 0.000600; visual box size=0.001200 0.001200 0.000600
- added link little_sensor_2_pad_057, mass 0.000001; collision box size=0.001200 0.001200 0.000600; visual box size=0.001200 0.001200 0.000600
- added link little_sensor_2_pad_058, mass 0.000001; collision box size=0.001200 0.001200 0.000600; visual box size=0.001200 0.001200 0.000600
- added link little_sensor_2_pad_059, mass 0.000001; collision box size=0.001200 0.001200 0.000600; visual box size=0.001200 0.001200 0.000600
- added link little_sensor_2_pad_060, mass 0.000001; collision box size=0.001200 0.001200 0.000600; visual box size=0.001200 0.001200 0.000600
- added link little_sensor_2_pad_061, mass 0.000001; collision box size=0.001200 0.001200 0.000600; visual box size=0.001200 0.001200 0.000600
- added link little_sensor_2_pad_062, mass 0.000001; collision box size=0.001200 0.001200 0.000600; visual box size=0.001200 0.001200 0.000600
- added link little_sensor_2_pad_063, mass 0.000001; collision box size=0.001200 0.001200 0.000600; visual box size=0.001200 0.001200 0.000600
- added link little_sensor_2_pad_064, mass 0.000001; collision box size=0.001200 0.001200 0.000600; visual box size=0.001200 0.001200 0.000600
- added link little_sensor_2_pad_065, mass 0.000001; collision box size=0.001200 0.001200 0.000600; visual box size=0.001200 0.001200 0.000600
- added link little_sensor_2_pad_066, mass 0.000001; collision box size=0.001200 0.001200 0.000600; visual box size=0.001200 0.001200 0.000600
- added link little_sensor_2_pad_067, mass 0.000001; collision box size=0.001200 0.001200 0.000600; visual box size=0.001200 0.001200 0.000600
- added link little_sensor_2_pad_068, mass 0.000001; collision box size=0.001200 0.001200 0.000600; visual box size=0.001200 0.001200 0.000600
- added link little_sensor_2_pad_069, mass 0.000001; collision box size=0.001200 0.001200 0.000600; visual box size=0.001200 0.001200 0.000600
- added link little_sensor_2_pad_070, mass 0.000001; collision box size=0.001200 0.001200 0.000600; visual box size=0.001200 0.001200 0.000600
- added link little_sensor_2_pad_071, mass 0.000001; collision box size=0.001200 0.001200 0.000600; visual box size=0.001200 0.001200 0.000600
- added link little_sensor_2_pad_072, mass 0.000001; collision box size=0.001200 0.001200 0.000600; visual box size=0.001200 0.001200 0.000600
- added link little_sensor_2_pad_073, mass 0.000001; collision box size=0.001200 0.001200 0.000600; visual box size=0.001200 0.001200 0.000600
- added link little_sensor_2_pad_074, mass 0.000001; collision box size=0.001200 0.001200 0.000600; visual box size=0.001200 0.001200 0.000600
- added link little_sensor_2_pad_075, mass 0.000001; collision box size=0.001200 0.001200 0.000600; visual box size=0.001200 0.001200 0.000600
- added link little_sensor_2_pad_076, mass 0.000001; collision box size=0.001200 0.001200 0.000600; visual box size=0.001200 0.001200 0.000600
- added link little_sensor_2_pad_077, mass 0.000001; collision box size=0.001200 0.001200 0.000600; visual box size=0.001200 0.001200 0.000600
- added link little_sensor_2_pad_078, mass 0.000001; collision box size=0.001200 0.001200 0.000600; visual box size=0.001200 0.001200 0.000600
- added link little_sensor_2_pad_079, mass 0.000001; collision box size=0.001200 0.001200 0.000600; visual box size=0.001200 0.001200 0.000600
- added link little_sensor_2_pad_080, mass 0.000001; collision box size=0.001200 0.001200 0.000600; visual box size=0.001200 0.001200 0.000600
Joints:
- added joint little_sensor_2_pad_001_joint: type fixed, parent little_force_sensor_2, child little_sensor_2_pad_001, origin xyz=-0.004200 -0.005400 0.000300 rpy=0 0 0
- added joint little_sensor_2_pad_002_joint: type fixed, parent little_force_sensor_2, child little_sensor_2_pad_002, origin xyz=-0.004200 -0.004200 0.000300 rpy=0 0 0
- added joint little_sensor_2_pad_003_joint: type fixed, parent little_force_sensor_2, child little_sensor_2_pad_003, origin xyz=-0.004200 -0.003000 0.000300 rpy=0 0 0
- added joint little_sensor_2_pad_004_joint: type fixed, parent little_force_sensor_2, child little_sensor_2_pad_004, origin xyz=-0.004200 -0.001800 0.000300 rpy=0 0 0
- added joint little_sensor_2_pad_005_joint: type fixed, parent little_force_sensor_2, child little_sensor_2_pad_005, origin xyz=-0.004200 -0.000600 0.000300 rpy=0 0 0
- added joint little_sensor_2_pad_006_joint: type fixed, parent little_force_sensor_2, child little_sensor_2_pad_006, origin xyz=-0.004200 0.000600 0.000300 rpy=0 0 0
- added joint little_sensor_2_pad_007_joint: type fixed, parent little_force_sensor_2, child little_sensor_2_pad_007, origin xyz=-0.004200 0.001800 0.000300 rpy=0 0 0
- added joint little_sensor_2_pad_008_joint: type fixed, parent little_force_sensor_2, child little_sensor_2_pad_008, origin xyz=-0.004200 0.003000 0.000300 rpy=0 0 0
- added joint little_sensor_2_pad_009_joint: type fixed, parent little_force_sensor_2, child little_sensor_2_pad_009, origin xyz=-0.004200 0.004200 0.000300 rpy=0 0 0
- added joint little_sensor_2_pad_010_joint: type fixed, parent little_force_sensor_2, child little_sensor_2_pad_010, origin xyz=-0.004200 0.005400 0.000300 rpy=0 0 0
- added joint little_sensor_2_pad_011_joint: type fixed, parent little_force_sensor_2, child little_sensor_2_pad_011, origin xyz=-0.003000 -0.005400 0.000300 rpy=0 0 0
- added joint little_sensor_2_pad_012_joint: type fixed, parent little_force_sensor_2, child little_sensor_2_pad_012, origin xyz=-0.003000 -0.004200 0.000300 rpy=0 0 0
- added joint little_sensor_2_pad_013_joint: type fixed, parent little_force_sensor_2, child little_sensor_2_pad_013, origin xyz=-0.003000 -0.003000 0.000300 rpy=0 0 0
- added joint little_sensor_2_pad_014_joint: type fixed, parent little_force_sensor_2, child little_sensor_2_pad_014, origin xyz=-0.003000 -0.001800 0.000300 rpy=0 0 0
- added joint little_sensor_2_pad_015_joint: type fixed, parent little_force_sensor_2, child little_sensor_2_pad_015, origin xyz=-0.003000 -0.000600 0.000300 rpy=0 0 0
- added joint little_sensor_2_pad_016_joint: type fixed, parent little_force_sensor_2, child little_sensor_2_pad_016, origin xyz=-0.003000 0.000600 0.000300 rpy=0 0 0
- added joint little_sensor_2_pad_017_joint: type fixed, parent little_force_sensor_2, child little_sensor_2_pad_017, origin xyz=-0.003000 0.001800 0.000300 rpy=0 0 0
- added joint little_sensor_2_pad_018_joint: type fixed, parent little_force_sensor_2, child little_sensor_2_pad_018, origin xyz=-0.003000 0.003000 0.000300 rpy=0 0 0
- added joint little_sensor_2_pad_019_joint: type fixed, parent little_force_sensor_2, child little_sensor_2_pad_019, origin xyz=-0.003000 0.004200 0.000300 rpy=0 0 0
- added joint little_sensor_2_pad_020_joint: type fixed, parent little_force_sensor_2, child little_sensor_2_pad_020, origin xyz=-0.003000 0.005400 0.000300 rpy=0 0 0
- added joint little_sensor_2_pad_021_joint: type fixed, parent little_force_sensor_2, child little_sensor_2_pad_021, origin xyz=-0.001800 -0.005400 0.000300 rpy=0 0 0
- added joint little_sensor_2_pad_022_joint: type fixed, parent little_force_sensor_2, child little_sensor_2_pad_022, origin xyz=-0.001800 -0.004200 0.000300 rpy=0 0 0
- added joint little_sensor_2_pad_023_joint: type fixed, parent little_force_sensor_2, child little_sensor_2_pad_023, origin xyz=-0.001800 -0.003000 0.000300 rpy=0 0 0
- added joint little_sensor_2_pad_024_joint: type fixed, parent little_force_sensor_2, child little_sensor_2_pad_024, origin xyz=-0.001800 -0.001800 0.000300 rpy=0 0 0
- added joint little_sensor_2_pad_025_joint: type fixed, parent little_force_sensor_2, child little_sensor_2_pad_025, origin xyz=-0.001800 -0.000600 0.000300 rpy=0 0 0
- added joint little_sensor_2_pad_026_joint: type fixed, parent little_force_sensor_2, child little_sensor_2_pad_026, origin xyz=-0.001800 0.000600 0.000300 rpy=0 0 0
- added joint little_sensor_2_pad_027_joint: type fixed, parent little_force_sensor_2, child little_sensor_2_pad_027, origin xyz=-0.001800 0.001800 0.000300 rpy=0 0 0
- added joint little_sensor_2_pad_028_joint: type fixed, parent little_force_sensor_2, child little_sensor_2_pad_028, origin xyz=-0.001800 0.003000 0.000300 rpy=0 0 0
- added joint little_sensor_2_pad_029_joint: type fixed, parent little_force_sensor_2, child little_sensor_2_pad_029, origin xyz=-0.001800 0.004200 0.000300 rpy=0 0 0
- added joint little_sensor_2_pad_030_joint: type fixed, parent little_force_sensor_2, child little_sensor_2_pad_030, origin xyz=-0.001800 0.005400 0.000300 rpy=0 0 0
- added joint little_sensor_2_pad_031_joint: type fixed, parent little_force_sensor_2, child little_sensor_2_pad_031, origin xyz=-0.000600 -0.005400 0.000300 rpy=0 0 0
- added joint little_sensor_2_pad_032_joint: type fixed, parent little_force_sensor_2, child little_sensor_2_pad_032, origin xyz=-0.000600 -0.004200 0.000300 rpy=0 0 0
- added joint little_sensor_2_pad_033_joint: type fixed, parent little_force_sensor_2, child little_sensor_2_pad_033, origin xyz=-0.000600 -0.003000 0.000300 rpy=0 0 0
- added joint little_sensor_2_pad_034_joint: type fixed, parent little_force_sensor_2, child little_sensor_2_pad_034, origin xyz=-0.000600 -0.001800 0.000300 rpy=0 0 0
- added joint little_sensor_2_pad_035_joint: type fixed, parent little_force_sensor_2, child little_sensor_2_pad_035, origin xyz=-0.000600 -0.000600 0.000300 rpy=0 0 0
- added joint little_sensor_2_pad_036_joint: type fixed, parent little_force_sensor_2, child little_sensor_2_pad_036, origin xyz=-0.000600 0.000600 0.000300 rpy=0 0 0
- added joint little_sensor_2_pad_037_joint: type fixed, parent little_force_sensor_2, child little_sensor_2_pad_037, origin xyz=-0.000600 0.001800 0.000300 rpy=0 0 0
- added joint little_sensor_2_pad_038_joint: type fixed, parent little_force_sensor_2, child little_sensor_2_pad_038, origin xyz=-0.000600 0.003000 0.000300 rpy=0 0 0
- added joint little_sensor_2_pad_039_joint: type fixed, parent little_force_sensor_2, child little_sensor_2_pad_039, origin xyz=-0.000600 0.004200 0.000300 rpy=0 0 0
- added joint little_sensor_2_pad_040_joint: type fixed, parent little_force_sensor_2, child little_sensor_2_pad_040, origin xyz=-0.000600 0.005400 0.000300 rpy=0 0 0
- added joint little_sensor_2_pad_041_joint: type fixed, parent little_force_sensor_2, child little_sensor_2_pad_041, origin xyz=0.000600 -0.005400 0.000300 rpy=0 0 0
- added joint little_sensor_2_pad_042_joint: type fixed, parent little_force_sensor_2, child little_sensor_2_pad_042, origin xyz=0.000600 -0.004200 0.000300 rpy=0 0 0
- added joint little_sensor_2_pad_043_joint: type fixed, parent little_force_sensor_2, child little_sensor_2_pad_043, origin xyz=0.000600 -0.003000 0.000300 rpy=0 0 0
- added joint little_sensor_2_pad_044_joint: type fixed, parent little_force_sensor_2, child little_sensor_2_pad_044, origin xyz=0.000600 -0.001800 0.000300 rpy=0 0 0
- added joint little_sensor_2_pad_045_joint: type fixed, parent little_force_sensor_2, child little_sensor_2_pad_045, origin xyz=0.000600 -0.000600 0.000300 rpy=0 0 0
- added joint little_sensor_2_pad_046_joint: type fixed, parent little_force_sensor_2, child little_sensor_2_pad_046, origin xyz=0.000600 0.000600 0.000300 rpy=0 0 0
- added joint little_sensor_2_pad_047_joint: type fixed, parent little_force_sensor_2, child little_sensor_2_pad_047, origin xyz=0.000600 0.001800 0.000300 rpy=0 0 0
- added joint little_sensor_2_pad_048_joint: type fixed, parent little_force_sensor_2, child little_sensor_2_pad_048, origin xyz=0.000600 0.003000 0.000300 rpy=0 0 0
- added joint little_sensor_2_pad_049_joint: type fixed, parent little_force_sensor_2, child little_sensor_2_pad_049, origin xyz=0.000600 0.004200 0.000300 rpy=0 0 0
- added joint little_sensor_2_pad_050_joint: type fixed, parent little_force_sensor_2, child little_sensor_2_pad_050, origin xyz=0.000600 0.005400 0.000300 rpy=0 0 0
- added joint little_sensor_2_pad_051_joint: type fixed, parent little_force_sensor_2, child little_sensor_2_pad_051, origin xyz=0.001800 -0.005400 0.000300 rpy=0 0 0
- added joint little_sensor_2_pad_052_joint: type fixed, parent little_force_sensor_2, child little_sensor_2_pad_052, origin xyz=0.001800 -0.004200 0.000300 rpy=0 0 0
- added joint little_sensor_2_pad_053_joint: type fixed, parent little_force_sensor_2, child little_sensor_2_pad_053, origin xyz=0.001800 -0.003000 0.000300 rpy=0 0 0
- added joint little_sensor_2_pad_054_joint: type fixed, parent little_force_sensor_2, child little_sensor_2_pad_054, origin xyz=0.001800 -0.001800 0.000300 rpy=0 0 0
- added joint little_sensor_2_pad_055_joint: type fixed, parent little_force_sensor_2, child little_sensor_2_pad_055, origin xyz=0.001800 -0.000600 0.000300 rpy=0 0 0
- added joint little_sensor_2_pad_056_joint: type fixed, parent little_force_sensor_2, child little_sensor_2_pad_056, origin xyz=0.001800 0.000600 0.000300 rpy=0 0 0
- added joint little_sensor_2_pad_057_joint: type fixed, parent little_force_sensor_2, child little_sensor_2_pad_057, origin xyz=0.001800 0.001800 0.000300 rpy=0 0 0
- added joint little_sensor_2_pad_058_joint: type fixed, parent little_force_sensor_2, child little_sensor_2_pad_058, origin xyz=0.001800 0.003000 0.000300 rpy=0 0 0
- added joint little_sensor_2_pad_059_joint: type fixed, parent little_force_sensor_2, child little_sensor_2_pad_059, origin xyz=0.001800 0.004200 0.000300 rpy=0 0 0
- added joint little_sensor_2_pad_060_joint: type fixed, parent little_force_sensor_2, child little_sensor_2_pad_060, origin xyz=0.001800 0.005400 0.000300 rpy=0 0 0
- added joint little_sensor_2_pad_061_joint: type fixed, parent little_force_sensor_2, child little_sensor_2_pad_061, origin xyz=0.003000 -0.005400 0.000300 rpy=0 0 0
- added joint little_sensor_2_pad_062_joint: type fixed, parent little_force_sensor_2, child little_sensor_2_pad_062, origin xyz=0.003000 -0.004200 0.000300 rpy=0 0 0
- added joint little_sensor_2_pad_063_joint: type fixed, parent little_force_sensor_2, child little_sensor_2_pad_063, origin xyz=0.003000 -0.003000 0.000300 rpy=0 0 0
- added joint little_sensor_2_pad_064_joint: type fixed, parent little_force_sensor_2, child little_sensor_2_pad_064, origin xyz=0.003000 -0.001800 0.000300 rpy=0 0 0
- added joint little_sensor_2_pad_065_joint: type fixed, parent little_force_sensor_2, child little_sensor_2_pad_065, origin xyz=0.003000 -0.000600 0.000300 rpy=0 0 0
- added joint little_sensor_2_pad_066_joint: type fixed, parent little_force_sensor_2, child little_sensor_2_pad_066, origin xyz=0.003000 0.000600 0.000300 rpy=0 0 0
- added joint little_sensor_2_pad_067_joint: type fixed, parent little_force_sensor_2, child little_sensor_2_pad_067, origin xyz=0.003000 0.001800 0.000300 rpy=0 0 0
- added joint little_sensor_2_pad_068_joint: type fixed, parent little_force_sensor_2, child little_sensor_2_pad_068, origin xyz=0.003000 0.003000 0.000300 rpy=0 0 0
- added joint little_sensor_2_pad_069_joint: type fixed, parent little_force_sensor_2, child little_sensor_2_pad_069, origin xyz=0.003000 0.004200 0.000300 rpy=0 0 0
- added joint little_sensor_2_pad_070_joint: type fixed, parent little_force_sensor_2, child little_sensor_2_pad_070, origin xyz=0.003000 0.005400 0.000300 rpy=0 0 0
- added joint little_sensor_2_pad_071_joint: type fixed, parent little_force_sensor_2, child little_sensor_2_pad_071, origin xyz=0.004200 -0.005400 0.000300 rpy=0 0 0
- added joint little_sensor_2_pad_072_joint: type fixed, parent little_force_sensor_2, child little_sensor_2_pad_072, origin xyz=0.004200 -0.004200 0.000300 rpy=0 0 0
- added joint little_sensor_2_pad_073_joint: type fixed, parent little_force_sensor_2, child little_sensor_2_pad_073, origin xyz=0.004200 -0.003000 0.000300 rpy=0 0 0
- added joint little_sensor_2_pad_074_joint: type fixed, parent little_force_sensor_2, child little_sensor_2_pad_074, origin xyz=0.004200 -0.001800 0.000300 rpy=0 0 0
- added joint little_sensor_2_pad_075_joint: type fixed, parent little_force_sensor_2, child little_sensor_2_pad_075, origin xyz=0.004200 -0.000600 0.000300 rpy=0 0 0
- added joint little_sensor_2_pad_076_joint: type fixed, parent little_force_sensor_2, child little_sensor_2_pad_076, origin xyz=0.004200 0.000600 0.000300 rpy=0 0 0
- added joint little_sensor_2_pad_077_joint: type fixed, parent little_force_sensor_2, child little_sensor_2_pad_077, origin xyz=0.004200 0.001800 0.000300 rpy=0 0 0
- added joint little_sensor_2_pad_078_joint: type fixed, parent little_force_sensor_2, child little_sensor_2_pad_078, origin xyz=0.004200 0.003000 0.000300 rpy=0 0 0
- added joint little_sensor_2_pad_079_joint: type fixed, parent little_force_sensor_2, child little_sensor_2_pad_079, origin xyz=0.004200 0.004200 0.000300 rpy=0 0 0
- added joint little_sensor_2_pad_080_joint: type fixed, parent little_force_sensor_2, child little_sensor_2_pad_080, origin xyz=0.004200 0.005400 0.000300 rpy=0 0 0
