Commit message: 🚀 Initial commit: Isaac Grasp Workspace
📊 Project Contents:
✅ cabinet_sensor_project/ - Complete project with 997 sensor pads
   - inspire_hand_with_sensors/ - Latest Inspire Hand (997 sensor pads)
   - franka_with_sensors/ - Franka robot integration
   - Comprehensive sensor configurations and scripts
   - Experimental data and analysis tools

🎯 Highlights:
- 17 force sensors with 997 total contact points
- Isaac Sim compatible USD files (21MB)
- Isaac Lab configurations
- Complete documentation and process guides
- Franka Panda integration
- Experimental scripts and analysis tools

🔧 Technical Specifications:
- URDF with all sensor definitions
- Isaac Sim 4.5+ compatible
- PhysX physics integration
- Contact sensor threshold: 15g (0.147N)
- Update rate: 200 FPS
- Uniform pad thickness: 0.6mm

📋 Excluded: IsaacLab/ (external dependency)

This workspace contains the complete tactile sensing research project
for the Inspire Hand with comprehensive Isaac Sim integration.

File: cabinet_sensor_project/inspire_hand_with_sensors/urdf/inspire_hand_processed_with_pads.urdf (robot description, URDF)
Before this commit: robot inspire_hand_with_sensors, 983 links, 982 joints
Links:
- added link index_sensor_3_pad_001, mass 0.000001; collision box size=0.001200 0.001200 0.000600; visual box size=0.001200 0.001200 0.000600
- added link index_sensor_3_pad_002, mass 0.000001; collision box size=0.001200 0.001200 0.000600; visual box size=0.001200 0.001200 0.000600
- added link index_sensor_3_pad_003, mass 0.000001; collision box size=0.001200 0.001200 0.000600; visual box size=0.001200 0.001200 0.000600
- added link index_sensor_3_pad_004, mass 0.000001; collision box size=0.001200 0.001200 0.000600; visual box size=0.001200 0.001200 0.000600
- added link index_sensor_3_pad_005, mass 0.000001; collision box size=0.001200 0.001200 0.000600; visual box size=0.001200 0.001200 0.000600
- added link index_sensor_3_pad_006, mass 0.000001; collision box size=0.001200 0.001200 0.000600; visual box size=0.001200 0.001200 0.000600
- added link index_sensor_3_pad_007, mass 0.000001; collision box size=0.001200 0.001200 0.000600; visual box size=0.001200 0.001200 0.000600
- added link index_sensor_3_pad_008, mass 0.000001; collision box size=0.001200 0.001200 0.000600; visual box size=0.001200 0.001200 0.000600
- added link index_sensor_3_pad_009, mass 0.000001; collision box size=0.001200 0.001200 0.000600; visual box size=0.001200 0.001200 0.000600
- added link little_sensor_3_pad_1, mass 1e-6; collision box size=0.001200 0.001200 0.000600; visual box size=0.001200 0.001200 0.000600
- added link little_sensor_3_pad_2, mass 1e-6; collision box size=0.001200 0.001200 0.000600; visual box size=0.001200 0.001200 0.000600
- added link little_sensor_3_pad_3, mass 1e-6; collision box size=0.001200 0.001200 0.000600; visual box size=0.001200 0.001200 0.000600
- added link little_sensor_3_pad_4, mass 1e-6; collision box size=0.001200 0.001200 0.000600; visual box size=0.001200 0.001200 0.000600
- added link little_sensor_3_pad_5, mass 1e-6; collision box size=0.001200 0.001200 0.000600; visual box size=0.001200 0.001200 0.000600
- added link little_sensor_3_pad_6, mass 1e-6; collision box size=0.001200 0.001200 0.000600; visual box size=0.001200 0.001200 0.000600
- added link little_sensor_3_pad_7, mass 1e-6; collision box size=0.001200 0.001200 0.000600; visual box size=0.001200 0.001200 0.000600
- added link little_sensor_3_pad_8, mass 1e-6; collision box size=0.001200 0.001200 0.000600; visual box size=0.001200 0.001200 0.000600
- added link little_sensor_3_pad_9, mass 1e-6; collision box size=0.001200 0.001200 0.000600; visual box size=0.001200 0.001200 0.000600
- added link middle_sensor_3_pad_001, mass 0.00001; collision box size=0.001200 0.001200 0.000600; visual box size=0.001200 0.001200 0.000600
- added link middle_sensor_3_pad_002, mass 0.00001; collision box size=0.001200 0.001200 0.000600; visual box size=0.001200 0.001200 0.000600
- added link middle_sensor_3_pad_003, mass 0.00001; collision box size=0.001200 0.001200 0.000600; visual box size=0.001200 0.001200 0.000600
- added link middle_sensor_3_pad_004, mass 0.00001; collision box size=0.001200 0.001200 0.000600; visual box size=0.001200 0.001200 0.000600
- added link middle_sensor_3_pad_005, mass 0.00001; collision box size=0.001200 0.001200 0.000600; visual box size=0.001200 0.001200 0.000600
- added link middle_sensor_3_pad_006, mass 0.00001; collision box size=0.001200 0.001200 0.000600; visual box size=0.001200 0.001200 0.000600
- added link middle_sensor_3_pad_007, mass 0.00001; collision box size=0.001200 0.001200 0.000600; visual box size=0.001200 0.001200 0.000600
- added link middle_sensor_3_pad_008, mass 0.00001; collision box size=0.001200 0.001200 0.000600; visual box size=0.001200 0.001200 0.000600
- added link middle_sensor_3_pad_009, mass 0.00001; collision box size=0.001200 0.001200 0.000600; visual box size=0.001200 0.001200 0.000600
- added link ring_sensor_3_pad_001, mass 0.00001; collision box size=0.001200 0.001200 0.000600; visual box size=0.001200 0.001200 0.000600
- added link ring_sensor_3_pad_002, mass 0.00001; collision box size=0.001200 0.001200 0.000600; visual box size=0.001200 0.001200 0.000600
- added link ring_sensor_3_pad_003, mass 0.00001; collision box size=0.001200 0.001200 0.000600; visual box size=0.001200 0.001200 0.000600
- added link ring_sensor_3_pad_004, mass 0.00001; collision box size=0.001200 0.001200 0.000600; visual box size=0.001200 0.001200 0.000600
- added link ring_sensor_3_pad_005, mass 0.00001; collision box size=0.001200 0.001200 0.000600; visual box size=0.001200 0.001200 0.000600
- added link ring_sensor_3_pad_006, mass 0.00001; collision box size=0.001200 0.001200 0.000600; visual box size=0.001200 0.001200 0.000600
- added link ring_sensor_3_pad_007, mass 0.00001; collision box size=0.001200 0.001200 0.000600; visual box size=0.001200 0.001200 0.000600
- added link ring_sensor_3_pad_008, mass 0.00001; collision box size=0.001200 0.001200 0.000600; visual box size=0.001200 0.001200 0.000600
- added link ring_sensor_3_pad_009, mass 0.00001; collision box size=0.001200 0.001200 0.000600; visual box size=0.001200 0.001200 0.000600
- added link thumb_sensor_4_pad_001, mass 0.000001; collision box size=0.001200 0.001200 0.000600; visual box size=0.001200 0.001200 0.000600
- added link thumb_sensor_4_pad_002, mass 0.000001; collision box size=0.001200 0.001200 0.000600; visual box size=0.001200 0.001200 0.000600
- added link thumb_sensor_4_pad_003, mass 0.000001; collision box size=0.001200 0.001200 0.000600; visual box size=0.001200 0.001200 0.000600
- added link thumb_sensor_4_pad_004, mass 0.000001; collision box size=0.001200 0.001200 0.000600; visual box size=0.001200 0.001200 0.000600
- added link thumb_sensor_4_pad_005, mass 0.000001; collision box size=0.001200 0.001200 0.000600; visual box size=0.001200 0.001200 0.000600
- added link thumb_sensor_4_pad_006, mass 0.000001; collision box size=0.001200 0.001200 0.000600; visual box size=0.001200 0.001200 0.000600
- added link thumb_sensor_4_pad_007, mass 0.000001; collision box size=0.001200 0.001200 0.000600; visual box size=0.001200 0.001200 0.000600
- added link thumb_sensor_4_pad_008, mass 0.000001; collision box size=0.001200 0.001200 0.000600; visual box size=0.001200 0.001200 0.000600
- added link thumb_sensor_4_pad_009, mass 0.000001; collision box size=0.001200 0.001200 0.000600; visual box size=0.001200 0.001200 0.000600
Joints:
- added joint index_sensor_3_pad_001_joint: type fixed, parent index_force_sensor_3, child index_sensor_3_pad_001, origin xyz=-0.001200 -0.001200 0.000300 rpy=0 0 0
- added joint index_sensor_3_pad_002_joint: type fixed, parent index_force_sensor_3, child index_sensor_3_pad_002, origin xyz=-0.001200 0.000000 0.000300 rpy=0 0 0
- added joint index_sensor_3_pad_003_joint: type fixed, parent index_force_sensor_3, child index_sensor_3_pad_003, origin xyz=-0.001200 0.001200 0.000300 rpy=0 0 0
- added joint index_sensor_3_pad_004_joint: type fixed, parent index_force_sensor_3, child index_sensor_3_pad_004, origin xyz=0.000000 -0.001200 0.000300 rpy=0 0 0
- added joint index_sensor_3_pad_005_joint: type fixed, parent index_force_sensor_3, child index_sensor_3_pad_005, origin xyz=0.000000 0.000000 0.000300 rpy=0 0 0
- added joint index_sensor_3_pad_006_joint: type fixed, parent index_force_sensor_3, child index_sensor_3_pad_006, origin xyz=0.000000 0.001200 0.000300 rpy=0 0 0
- added joint index_sensor_3_pad_007_joint: type fixed, parent index_force_sensor_3, child index_sensor_3_pad_007, origin xyz=0.001200 -0.001200 0.000300 rpy=0 0 0
- added joint index_sensor_3_pad_008_joint: type fixed, parent index_force_sensor_3, child index_sensor_3_pad_008, origin xyz=0.001200 0.000000 0.000300 rpy=0 0 0
- added joint index_sensor_3_pad_009_joint: type fixed, parent index_force_sensor_3, child index_sensor_3_pad_009, origin xyz=0.001200 0.001200 0.000300 rpy=0 0 0
- added joint little_sensor_3_pad_1_joint: type fixed, parent little_force_sensor_3, child little_sensor_3_pad_1, origin xyz=-0.001200 -0.001200 0.000300 rpy=0 0 0
- added joint little_sensor_3_pad_2_joint: type fixed, parent little_force_sensor_3, child little_sensor_3_pad_2, origin xyz=-0.001200 0.000000 0.000300 rpy=0 0 0
- added joint little_sensor_3_pad_3_joint: type fixed, parent little_force_sensor_3, child little_sensor_3_pad_3, origin xyz=-0.001200 0.001200 0.000300 rpy=0 0 0
- added joint little_sensor_3_pad_4_joint: type fixed, parent little_force_sensor_3, child little_sensor_3_pad_4, origin xyz=0.000000 -0.001200 0.000300 rpy=0 0 0
- added joint little_sensor_3_pad_5_joint: type fixed, parent little_force_sensor_3, child little_sensor_3_pad_5, origin xyz=0.000000 0.000000 0.000300 rpy=0 0 0
- added joint little_sensor_3_pad_6_joint: type fixed, parent little_force_sensor_3, child little_sensor_3_pad_6, origin xyz=0.000000 0.001200 0.000300 rpy=0 0 0
- added joint little_sensor_3_pad_7_joint: type fixed, parent little_force_sensor_3, child little_sensor_3_pad_7, origin xyz=0.001200 -0.001200 0.000300 rpy=0 0 0
- added joint little_sensor_3_pad_8_joint: type fixed, parent little_force_sensor_3, child little_sensor_3_pad_8, origin xyz=0.001200 0.000000 0.000300 rpy=0 0 0
- added joint little_sensor_3_pad_9_joint: type fixed, parent little_force_sensor_3, child little_sensor_3_pad_9, origin xyz=0.001200 0.001200 0.000300 rpy=0 0 0
- added joint middle_sensor_3_pad_001_joint: type fixed, parent middle_force_sensor_3, child middle_sensor_3_pad_001, origin xyz=-0.001200 -0.001200 0.000300 rpy=0 0 0
- added joint middle_sensor_3_pad_002_joint: type fixed, parent middle_force_sensor_3, child middle_sensor_3_pad_002, origin xyz=-0.001200 0.000000 0.000300 rpy=0 0 0
- added joint middle_sensor_3_pad_003_joint: type fixed, parent middle_force_sensor_3, child middle_sensor_3_pad_003, origin xyz=-0.001200 0.001200 0.000300 rpy=0 0 0
- added joint middle_sensor_3_pad_004_joint: type fixed, parent middle_force_sensor_3, child middle_sensor_3_pad_004, origin xyz=0.000000 -0.001200 0.000300 rpy=0 0 0
- added joint middle_sensor_3_pad_005_joint: type fixed, parent middle_force_sensor_3, child middle_sensor_3_pad_005, origin xyz=0.000000 0.000000 0.000300 rpy=0 0 0
- added joint middle_sensor_3_pad_006_joint: type fixed, parent middle_force_sensor_3, child middle_sensor_3_pad_006, origin xyz=0.000000 0.001200 0.000300 rpy=0 0 0
- added joint middle_sensor_3_pad_007_joint: type fixed, parent middle_force_sensor_3, child middle_sensor_3_pad_007, origin xyz=0.001200 -0.001200 0.000300 rpy=0 0 0
- added joint middle_sensor_3_pad_008_joint: type fixed, parent middle_force_sensor_3, child middle_sensor_3_pad_008, origin xyz=0.001200 0.000000 0.000300 rpy=0 0 0
- added joint middle_sensor_3_pad_009_joint: type fixed, parent middle_force_sensor_3, child middle_sensor_3_pad_009, origin xyz=0.001200 0.001200 0.000300 rpy=0 0 0
- added joint ring_sensor_3_pad_001_joint: type fixed, parent ring_force_sensor_3, child ring_sensor_3_pad_001, origin xyz=-0.001200 -0.001200 0.000300 rpy=0 0 0
- added joint ring_sensor_3_pad_002_joint: type fixed, parent ring_force_sensor_3, child ring_sensor_3_pad_002, origin xyz=-0.001200 0.000000 0.000300 rpy=0 0 0
- added joint ring_sensor_3_pad_003_joint: type fixed, parent ring_force_sensor_3, child ring_sensor_3_pad_003, origin xyz=-0.001200 0.001200 0.000300 rpy=0 0 0
- added joint ring_sensor_3_pad_004_joint: type fixed, parent ring_force_sensor_3, child ring_sensor_3_pad_004, origin xyz=0.000000 -0.001200 0.000300 rpy=0 0 0
- added joint ring_sensor_3_pad_005_joint: type fixed, parent ring_force_sensor_3, child ring_sensor_3_pad_005, origin xyz=0.000000 0.000000 0.000300 rpy=0 0 0
- added joint ring_sensor_3_pad_006_joint: type fixed, parent ring_force_sensor_3, child ring_sensor_3_pad_006, origin xyz=0.000000 0.001200 0.000300 rpy=0 0 0
- added joint ring_sensor_3_pad_007_joint: type fixed, parent ring_force_sensor_3, child ring_sensor_3_pad_007, origin xyz=0.001200 -0.001200 0.000300 rpy=0 0 0
- added joint ring_sensor_3_pad_008_joint: type fixed, parent ring_force_sensor_3, child ring_sensor_3_pad_008, origin xyz=0.001200 0.000000 0.000300 rpy=0 0 0
- added joint ring_sensor_3_pad_009_joint: type fixed, parent ring_force_sensor_3, child ring_sensor_3_pad_009, origin xyz=0.001200 0.001200 0.000300 rpy=0 0 0
- added joint thumb_sensor_4_pad_001_joint: type fixed, parent thumb_force_sensor_4, child thumb_sensor_4_pad_001, origin xyz=-0.001200 -0.001200 0.000300 rpy=0 0 0
- added joint thumb_sensor_4_pad_002_joint: type fixed, parent thumb_force_sensor_4, child thumb_sensor_4_pad_002, origin xyz=-0.001200 0.000000 0.000300 rpy=0 0 0
- added joint thumb_sensor_4_pad_003_joint: type fixed, parent thumb_force_sensor_4, child thumb_sensor_4_pad_003, origin xyz=-0.001200 0.001200 0.000300 rpy=0 0 0
- added joint thumb_sensor_4_pad_004_joint: type fixed, parent thumb_force_sensor_4, child thumb_sensor_4_pad_004, origin xyz=0.000000 -0.001200 0.000300 rpy=0 0 0
- added joint thumb_sensor_4_pad_005_joint: type fixed, parent thumb_force_sensor_4, child thumb_sensor_4_pad_005, origin xyz=0.000000 0.000000 0.000300 rpy=0 0 0
- added joint thumb_sensor_4_pad_006_joint: type fixed, parent thumb_force_sensor_4, child thumb_sensor_4_pad_006, origin xyz=0.000000 0.001200 0.000300 rpy=0 0 0
- added joint thumb_sensor_4_pad_007_joint: type fixed, parent thumb_force_sensor_4, child thumb_sensor_4_pad_007, origin xyz=0.001200 -0.001200 0.000300 rpy=0 0 0
- added joint thumb_sensor_4_pad_008_joint: type fixed, parent thumb_force_sensor_4, child thumb_sensor_4_pad_008, origin xyz=0.001200 0.000000 0.000300 rpy=0 0 0
- added joint thumb_sensor_4_pad_009_joint: type fixed, parent thumb_force_sensor_4, child thumb_sensor_4_pad_009, origin xyz=0.001200 0.001200 0.000300 rpy=0 0 0
