Commit message: Add middle_force_sensor_3 pads: 970 total sensor pads
✨ New Features:
- Added 9 new sensor pads to middle_force_sensor_3 (3×3 layout)
- Total sensor pads: 970 (was 961)
- USD conversion script for Isaac Sim 4.5

🛠️ Technical Details:
- Pad size: 1.2×1.2×0.6mm (consistent with other finger sensors)
- Color: Cyan (matches other middle sensors)
- Successfully converted URDF to USD (20.95 MB)

📁 Files Added/Modified:
- urdf/inspire_hand_processed_with_pads.urdf (updated)
- convert_urdf_to_usd_with_middle3_pads.py (new)
- usd/inspire_hand_processed_with_pads.usd (updated)
- README_SENSOR_PAD_PROCESS.md (updated)

File: urdf/inspire_hand_processed_with_pads.urdf (robot description, URDF)
Before this commit: robot inspire_hand_with_sensors, 992 links, 991 joints
Links:
- added link middle_sensor_3_pad_001, mass 0.00001; collision box size=0.001200 0.001200 0.000600; visual box size=0.001200 0.001200 0.000600
- added link middle_sensor_3_pad_002, mass 0.00001; collision box size=0.001200 0.001200 0.000600; visual box size=0.001200 0.001200 0.000600
- added link middle_sensor_3_pad_003, mass 0.00001; collision box size=0.001200 0.001200 0.000600; visual box size=0.001200 0.001200 0.000600
- added link middle_sensor_3_pad_004, mass 0.00001; collision box size=0.001200 0.001200 0.000600; visual box size=0.001200 0.001200 0.000600
- added link middle_sensor_3_pad_005, mass 0.00001; collision box size=0.001200 0.001200 0.000600; visual box size=0.001200 0.001200 0.000600
- added link middle_sensor_3_pad_006, mass 0.00001; collision box size=0.001200 0.001200 0.000600; visual box size=0.001200 0.001200 0.000600
- added link middle_sensor_3_pad_007, mass 0.00001; collision box size=0.001200 0.001200 0.000600; visual box size=0.001200 0.001200 0.000600
- added link middle_sensor_3_pad_008, mass 0.00001; collision box size=0.001200 0.001200 0.000600; visual box size=0.001200 0.001200 0.000600
- added link middle_sensor_3_pad_009, mass 0.00001; collision box size=0.001200 0.001200 0.000600; visual box size=0.001200 0.001200 0.000600
Joints:
- added joint middle_sensor_3_pad_001_joint: type fixed, parent middle_force_sensor_3, child middle_sensor_3_pad_001, origin xyz=-0.001200 -0.001200 0.000300 rpy=0 0 0
- added joint middle_sensor_3_pad_002_joint: type fixed, parent middle_force_sensor_3, child middle_sensor_3_pad_002, origin xyz=-0.001200 0.000000 0.000300 rpy=0 0 0
- added joint middle_sensor_3_pad_003_joint: type fixed, parent middle_force_sensor_3, child middle_sensor_3_pad_003, origin xyz=-0.001200 0.001200 0.000300 rpy=0 0 0
- added joint middle_sensor_3_pad_004_joint: type fixed, parent middle_force_sensor_3, child middle_sensor_3_pad_004, origin xyz=0.000000 -0.001200 0.000300 rpy=0 0 0
- added joint middle_sensor_3_pad_005_joint: type fixed, parent middle_force_sensor_3, child middle_sensor_3_pad_005, origin xyz=0.000000 0.000000 0.000300 rpy=0 0 0
- added joint middle_sensor_3_pad_006_joint: type fixed, parent middle_force_sensor_3, child middle_sensor_3_pad_006, origin xyz=0.000000 0.001200 0.000300 rpy=0 0 0
- added joint middle_sensor_3_pad_007_joint: type fixed, parent middle_force_sensor_3, child middle_sensor_3_pad_007, origin xyz=0.001200 -0.001200 0.000300 rpy=0 0 0
- added joint middle_sensor_3_pad_008_joint: type fixed, parent middle_force_sensor_3, child middle_sensor_3_pad_008, origin xyz=0.001200 0.000000 0.000300 rpy=0 0 0
- added joint middle_sensor_3_pad_009_joint: type fixed, parent middle_force_sensor_3, child middle_sensor_3_pad_009, origin xyz=0.001200 0.001200 0.000300 rpy=0 0 0

Commit message: Add ring_force_sensor_3 pads: 979 total sensor pads
✨ New Features:
- Added 9 new sensor pads to ring_force_sensor_3 (3×3 layout)
- Total sensor pads: 979 (was 970)
- Updated USD conversion script for ring_sensor_3

🛠️ Technical Details:
- Pad size: 1.2×1.2×0.6mm (consistent with other finger sensors)
- Color: Magenta (matches other ring sensors)
- Successfully converted URDF to USD (20.95 MB)

📁 Files Modified:
- urdf/inspire_hand_processed_with_pads.urdf (updated)
- convert_urdf_to_usd_with_ring3_pads.py (new)
- README.md (sensor count updated to 979)
- usd/inspire_hand_processed_with_pads.usd (updated)

File: urdf/inspire_hand_processed_with_pads.urdf (robot description, URDF)
Before this commit: robot inspire_hand_with_sensors, 1001 links, 1000 joints
Links:
- added link ring_sensor_3_pad_001, mass 0.00001; collision box size=0.001200 0.001200 0.000600; visual box size=0.001200 0.001200 0.000600
- added link ring_sensor_3_pad_002, mass 0.00001; collision box size=0.001200 0.001200 0.000600; visual box size=0.001200 0.001200 0.000600
- added link ring_sensor_3_pad_003, mass 0.00001; collision box size=0.001200 0.001200 0.000600; visual box size=0.001200 0.001200 0.000600
- added link ring_sensor_3_pad_004, mass 0.00001; collision box size=0.001200 0.001200 0.000600; visual box size=0.001200 0.001200 0.000600
- added link ring_sensor_3_pad_005, mass 0.00001; collision box size=0.001200 0.001200 0.000600; visual box size=0.001200 0.001200 0.000600
- added link ring_sensor_3_pad_006, mass 0.00001; collision box size=0.001200 0.001200 0.000600; visual box size=0.001200 0.001200 0.000600
- added link ring_sensor_3_pad_007, mass 0.00001; collision box size=0.001200 0.001200 0.000600; visual box size=0.001200 0.001200 0.000600
- added link ring_sensor_3_pad_008, mass 0.00001; collision box size=0.001200 0.001200 0.000600; visual box size=0.001200 0.001200 0.000600
- added link ring_sensor_3_pad_009, mass 0.00001; collision box size=0.001200 0.001200 0.000600; visual box size=0.001200 0.001200 0.000600
Joints:
- added joint ring_sensor_3_pad_001_joint: type fixed, parent ring_force_sensor_3, child ring_sensor_3_pad_001, origin xyz=-0.001200 -0.001200 0.000300 rpy=0 0 0
- added joint ring_sensor_3_pad_002_joint: type fixed, parent ring_force_sensor_3, child ring_sensor_3_pad_002, origin xyz=-0.001200 0.000000 0.000300 rpy=0 0 0
- added joint ring_sensor_3_pad_003_joint: type fixed, parent ring_force_sensor_3, child ring_sensor_3_pad_003, origin xyz=-0.001200 0.001200 0.000300 rpy=0 0 0
- added joint ring_sensor_3_pad_004_joint: type fixed, parent ring_force_sensor_3, child ring_sensor_3_pad_004, origin xyz=0.000000 -0.001200 0.000300 rpy=0 0 0
- added joint ring_sensor_3_pad_005_joint: type fixed, parent ring_force_sensor_3, child ring_sensor_3_pad_005, origin xyz=0.000000 0.000000 0.000300 rpy=0 0 0
- added joint ring_sensor_3_pad_006_joint: type fixed, parent ring_force_sensor_3, child ring_sensor_3_pad_006, origin xyz=0.000000 0.001200 0.000300 rpy=0 0 0
- added joint ring_sensor_3_pad_007_joint: type fixed, parent ring_force_sensor_3, child ring_sensor_3_pad_007, origin xyz=0.001200 -0.001200 0.000300 rpy=0 0 0
- added joint ring_sensor_3_pad_008_joint: type fixed, parent ring_force_sensor_3, child ring_sensor_3_pad_008, origin xyz=0.001200 0.000000 0.000300 rpy=0 0 0
- added joint ring_sensor_3_pad_009_joint: type fixed, parent ring_force_sensor_3, child ring_sensor_3_pad_009, origin xyz=0.001200 0.001200 0.000300 rpy=0 0 0

Commit message: Update inspire hand configuration and add sensor processing files
- Updated inspire_hand_processed_with_pads.yaml configuration
- Modified inspire_hand_processed_with_pads.urdf
- Added convert_urdf_to_usd_with_little3_pads.py for URDF to USD conversion
- Added little_sensor_3_pads.xml sensor configuration

File: urdf/inspire_hand_processed_with_pads.urdf (robot description, URDF)
Before this commit: robot inspire_hand_with_sensors, 1010 links, 1009 joints
Links:
- added link little_sensor_3_pad_1, mass 1e-6; collision box size=0.001200 0.001200 0.000600; visual box size=0.001200 0.001200 0.000600
- added link little_sensor_3_pad_2, mass 1e-6; collision box size=0.001200 0.001200 0.000600; visual box size=0.001200 0.001200 0.000600
- added link little_sensor_3_pad_3, mass 1e-6; collision box size=0.001200 0.001200 0.000600; visual box size=0.001200 0.001200 0.000600
- added link little_sensor_3_pad_4, mass 1e-6; collision box size=0.001200 0.001200 0.000600; visual box size=0.001200 0.001200 0.000600
- added link little_sensor_3_pad_5, mass 1e-6; collision box size=0.001200 0.001200 0.000600; visual box size=0.001200 0.001200 0.000600
- added link little_sensor_3_pad_6, mass 1e-6; collision box size=0.001200 0.001200 0.000600; visual box size=0.001200 0.001200 0.000600
- added link little_sensor_3_pad_7, mass 1e-6; collision box size=0.001200 0.001200 0.000600; visual box size=0.001200 0.001200 0.000600
- added link little_sensor_3_pad_8, mass 1e-6; collision box size=0.001200 0.001200 0.000600; visual box size=0.001200 0.001200 0.000600
- added link little_sensor_3_pad_9, mass 1e-6; collision box size=0.001200 0.001200 0.000600; visual box size=0.001200 0.001200 0.000600
Joints:
- added joint little_sensor_3_pad_1_joint: type fixed, parent little_force_sensor_3, child little_sensor_3_pad_1, origin xyz=-0.001200 -0.001200 0.000300 rpy=0 0 0
- added joint little_sensor_3_pad_2_joint: type fixed, parent little_force_sensor_3, child little_sensor_3_pad_2, origin xyz=-0.001200 0.000000 0.000300 rpy=0 0 0
- added joint little_sensor_3_pad_3_joint: type fixed, parent little_force_sensor_3, child little_sensor_3_pad_3, origin xyz=-0.001200 0.001200 0.000300 rpy=0 0 0
- added joint little_sensor_3_pad_4_joint: type fixed, parent little_force_sensor_3, child little_sensor_3_pad_4, origin xyz=0.000000 -0.001200 0.000300 rpy=0 0 0
- added joint little_sensor_3_pad_5_joint: type fixed, parent little_force_sensor_3, child little_sensor_3_pad_5, origin xyz=0.000000 0.000000 0.000300 rpy=0 0 0
- added joint little_sensor_3_pad_6_joint: type fixed, parent little_force_sensor_3, child little_sensor_3_pad_6, origin xyz=0.000000 0.001200 0.000300 rpy=0 0 0
- added joint little_sensor_3_pad_7_joint: type fixed, parent little_force_sensor_3, child little_sensor_3_pad_7, origin xyz=0.001200 -0.001200 0.000300 rpy=0 0 0
- added joint little_sensor_3_pad_8_joint: type fixed, parent little_force_sensor_3, child little_sensor_3_pad_8, origin xyz=0.001200 0.000000 0.000300 rpy=0 0 0
- added joint little_sensor_3_pad_9_joint: type fixed, parent little_force_sensor_3, child little_sensor_3_pad_9, origin xyz=0.001200 0.001200 0.000300 rpy=0 0 0

Commit message: 🚀 Major Update: Add Thumb4 sensor and complete documentation
✨ New Features:
- Added thumb_force_sensor_4 with 9 pads (3×3 layout)
- Updated total sensor count: 979 → 997 pads
- Generated new USD file with all 997 sensors (21.0MB)
- Created thumb4-specific conversion script

�� Sensor Statistics:
- Total sensors: 17 (all force sensors covered)
- Total contact points: 997 tactile sensor pads
- New Thumb4: 9 pads, 1.2×1.2×0.6mm, white color

📝 Documentation Updates:
- Updated README.md with complete sensor distribution
- Refreshed README_SENSOR_PAD_PROCESS.md with full methodology
- Added detailed project structure and usage instructions
- Updated Isaac Lab configuration for all sensors

🔧 Technical Improvements:
- Validated URDF XML syntax with 997 pads
- Successful Isaac Sim conversion and USD export
- Isaac Lab YAML configuration updated
- All conversion scripts available

Files changed:
- urdf/inspire_hand_processed_with_pads.urdf (997 pads)
- usd/inspire_hand_processed_with_pads.usd (21.0MB)
- config/inspire_hand_processed_with_pads.yaml (17 sensors)
- convert_urdf_to_usd_with_thumb4_pads.py (new)
- thumb_sensor_4_pads.xml (new)
- README.md (updated)
- README_SENSOR_PAD_PROCESS.md (updated)

File: urdf/inspire_hand_processed_with_pads.urdf (robot description, URDF)
Before this commit: robot inspire_hand_with_sensors, 1019 links, 1018 joints
Links:
- added link thumb_sensor_4_pad_001, mass 0.000001; collision box size=0.001200 0.001200 0.000600; visual box size=0.001200 0.001200 0.000600
- added link thumb_sensor_4_pad_002, mass 0.000001; collision box size=0.001200 0.001200 0.000600; visual box size=0.001200 0.001200 0.000600
- added link thumb_sensor_4_pad_003, mass 0.000001; collision box size=0.001200 0.001200 0.000600; visual box size=0.001200 0.001200 0.000600
- added link thumb_sensor_4_pad_004, mass 0.000001; collision box size=0.001200 0.001200 0.000600; visual box size=0.001200 0.001200 0.000600
- added link thumb_sensor_4_pad_005, mass 0.000001; collision box size=0.001200 0.001200 0.000600; visual box size=0.001200 0.001200 0.000600
- added link thumb_sensor_4_pad_006, mass 0.000001; collision box size=0.001200 0.001200 0.000600; visual box size=0.001200 0.001200 0.000600
- added link thumb_sensor_4_pad_007, mass 0.000001; collision box size=0.001200 0.001200 0.000600; visual box size=0.001200 0.001200 0.000600
- added link thumb_sensor_4_pad_008, mass 0.000001; collision box size=0.001200 0.001200 0.000600; visual box size=0.001200 0.001200 0.000600
- added link thumb_sensor_4_pad_009, mass 0.000001; collision box size=0.001200 0.001200 0.000600; visual box size=0.001200 0.001200 0.000600
Joints:
- added joint thumb_sensor_4_pad_001_joint: type fixed, parent thumb_force_sensor_4, child thumb_sensor_4_pad_001, origin xyz=-0.001200 -0.001200 0.000300 rpy=0 0 0
- added joint thumb_sensor_4_pad_002_joint: type fixed, parent thumb_force_sensor_4, child thumb_sensor_4_pad_002, origin xyz=-0.001200 0.000000 0.000300 rpy=0 0 0
- added joint thumb_sensor_4_pad_003_joint: type fixed, parent thumb_force_sensor_4, child thumb_sensor_4_pad_003, origin xyz=-0.001200 0.001200 0.000300 rpy=0 0 0
- added joint thumb_sensor_4_pad_004_joint: type fixed, parent thumb_force_sensor_4, child thumb_sensor_4_pad_004, origin xyz=0.000000 -0.001200 0.000300 rpy=0 0 0
- added joint thumb_sensor_4_pad_005_joint: type fixed, parent thumb_force_sensor_4, child thumb_sensor_4_pad_005, origin xyz=0.000000 0.000000 0.000300 rpy=0 0 0
- added joint thumb_sensor_4_pad_006_joint: type fixed, parent thumb_force_sensor_4, child thumb_sensor_4_pad_006, origin xyz=0.000000 0.001200 0.000300 rpy=0 0 0
- added joint thumb_sensor_4_pad_007_joint: type fixed, parent thumb_force_sensor_4, child thumb_sensor_4_pad_007, origin xyz=0.001200 -0.001200 0.000300 rpy=0 0 0
- added joint thumb_sensor_4_pad_008_joint: type fixed, parent thumb_force_sensor_4, child thumb_sensor_4_pad_008, origin xyz=0.001200 0.000000 0.000300 rpy=0 0 0
- added joint thumb_sensor_4_pad_009_joint: type fixed, parent thumb_force_sensor_4, child thumb_sensor_4_pad_009, origin xyz=0.001200 0.001200 0.000300 rpy=0 0 0
